File: micromouse.kicad_pcb (KiCad board)
At the start: 2 copper layers, 8 parts, among them U1 STM32F103C8Tx, U2 L298N, U3 MPU-6050, U6 LM2596S-5, U7 LM2596S-3.3

Commit message: cap nhat pcb
Parts:
- removed DS1: OLED-128O064D, Display:OLED-128O064D
- removed U2: L298N, Package_TO_SOT_THT:TO-220-15_P2.54x5.08mm_StaggerOdd_Lead4.58mm_Vertical
- removed U3: MPU-6050, Sensor_Motion:InvenSense_QFN-24_4x4mm_P0.5mm
- removed U7: LM2596S-3.3, Package_TO_SOT_SMD:TO-263-5_TabPin3
- added C1: 220uF, Capacitor_Tantalum_SMD:CP_EIA-7343-31_Kemet-D_HandSolder, F.Cu at (158.3, 172.2)
- added C10: 100nF, Capacitor_SMD:C_0603_1608Metric, F.Cu at (169.0, 84.8)
- added C11: 1nF, Capacitor_SMD:C_0603_1608Metric, F.Cu at (198.5, 81.3)
- added C12: 1uF, Capacitor_SMD:C_0603_1608Metric, F.Cu at (198.5, 83.8)
- added C13: 100uF, Capacitor_SMD:C_0603_1608Metric, F.Cu at (103.8, 113.5)
- added C14: 10uF, Capacitor_SMD:C_0603_1608Metric, F.Cu at (208.3, 102.8)
- added C17: 100nF, Capacitor_SMD:C_0603_1608Metric, F.Cu at (162.5, 71.8)
- added C18: 0.1uF, Capacitor_SMD:C_0603_1608Metric, F.Cu at (161.0, 150.5)
- added C19: 0.1uF, Capacitor_SMD:C_0603_1608Metric, F.Cu at (192.5, 150.8)
- added C2: 100uF, Capacitor_Tantalum_SMD:CP_EIA-6032-28_Kemet-C_HandSolder, F.Cu at (100.7, 184.7)
- added C20: 22pF, Capacitor_SMD:C_0603_1608Metric, F.Cu at (157.5, 95.3)
- added C21: 22pF, Capacitor_SMD:C_0603_1608Metric, F.Cu at (157.5, 97.8)
- added C3: 10uF, Capacitor_Tantalum_SMD:CP_EIA-6032-28_Kemet-C_HandSolder, F.Cu at (154.9, 143.0)
- added C4: 10uF, Capacitor_Tantalum_SMD:CP_EIA-6032-28_Kemet-C_HandSolder, F.Cu at (184.0, 155.1)
- added C5: 100nF, Capacitor_SMD:C_0603_1608Metric, F.Cu at (156.4, 84.8)
- added C6: 100nF, Capacitor_SMD:C_0603_1608Metric, F.Cu at (159.0, 84.8)
- added C7: 100nF, Capacitor_SMD:C_0603_1608Metric, F.Cu at (161.5, 84.8)
- added C8: 100nF, Capacitor_SMD:C_0603_1608Metric, F.Cu at (164.0, 84.8)
- added C9: 10uF, Capacitor_SMD:C_0603_1608Metric, F.Cu at (166.5, 84.8)
- added D3: LED2, LED_SMD:LED_0603_1608Metric_Pad1.05x0.95mm_HandSolder, F.Cu at (197.6, 115.9)
- added FB1: FerriteBead, Ferrite_THT:LairdTech_28C0236-0JW-10, F.Cu at (188.4, 81.3)
- added J1: Conn_01x04_Pin, Connector_PinHeader_2.54mm:PinHeader_1x04_P2.54mm_Vertical, F.Cu at (92.5, 88.5)
- added J1: Conn_01x06_Pin, Connector_PinHeader_2.54mm:PinHeader_1x06_P2.54mm_Vertical, F.Cu at (123.2, 90.2)
- added J10: Conn_01x04_Pin, Connector_PinHeader_2.54mm:PinHeader_1x04_P2.54mm_Vertical, F.Cu at (260.0, 94.0)
- added J2: Conn_01x03_Pin, Connector_PinHeader_2.54mm:PinHeader_1x03_P2.54mm_Vertical, F.Cu at (261.0, 54.0)
- added J4: Conn_01x03_Pin, Connector_PinHeader_2.54mm:PinHeader_1x03_P2.54mm_Vertical, F.Cu at (184.5, 44.2)
- added J5: Conn_01x03_Pin, Connector_PinHeader_2.54mm:PinHeader_1x03_P2.54mm_Vertical, F.Cu at (105.0, 57.7)
- added J6: Conn_01x04_Pin, Connector_PinHeader_2.54mm:PinHeader_1x04_P2.54mm_Vertical, F.Cu at (246.5, 130.7)
- added J7: Conn_01x04_Pin, Connector_PinHeader_2.54mm:PinHeader_1x04_P2.54mm_Vertical, F.Cu at (239.5, 160.2)
- added J8: Conn_01x08_Pin, Connector_PinHeader_2.54mm:PinHeader_1x08_P2.54mm_Vertical, F.Cu at (192.4, 188.5)
- added J9: Conn_01x04, Connector_PinHeader_2.54mm:PinHeader_1x04_P2.54mm_Vertical, F.Cu at (97.0, 113.9)
- added L1: 33uH, Inductor_SMD:L_10.4x10.4_H4.8, F.Cu at (141.0, 175.5)
- added R3: 1M, Resistor_SMD:R_0805_2012Metric_Pad1.20x1.40mm_HandSolder, F.Cu at (162.7, 100.3)
- added R4: 10K, Resistor_SMD:R_0805_2012Metric_Pad1.20x1.40mm_HandSolder, F.Cu at (190.0, 111.3)
- added R5: 2K2, Resistor_SMD:R_0805_2012Metric_Pad1.20x1.40mm_HandSolder, F.Cu at (190.0, 114.2)
- added R6: 10K, Resistor_SMD:R_0805_2012Metric_Pad1.20x1.40mm_HandSolder, F.Cu at (190.0, 117.2)
- added R7: 2K2, Resistor_SMD:R_0805_2012Metric_Pad1.20x1.40mm_HandSolder, F.Cu at (190.0, 120.1)
- added SW1: SW_Push, Button_Switch_THT:SW_PUSH-12mm, F.Cu at (140.2, 69.8)
- added SW2: SW_Push, Button_Switch_THT:SW_PUSH-12mm, F.Cu at (188.7, 96.8)
- added U9: LM1117DT-3.3, Package_TO_SOT_SMD:TO-252-3_TabPin2, F.Cu at (172.4, 150.5)
- added Y1: 8MHz, Crystal:Crystal_SMD_HC49-SD_HandSoldering, F.Cu at (149.5, 98.2)
- D2: value 1N5822 -> LED1; footprint Diode_THT:D_DO-201AD_P15.24mm_Horizontal -> LED_SMD:LED_0603_1608Metric_Pad1.05x0.95mm_HandSolder
- moved U6 125.3 mm to (121.2, 178.0)
- moved D2 119.7 mm to (197.6, 113.3)
- moved U1 107.8 mm to (173.8, 96.0)
- moved D1 93.9 mm to (116.7, 167.5)
Connections:
- net /IROUT1 renamed /PA10
- net /IROUT2 renamed /PA11
- net /IROUT3 renamed /PA12
- net /OLED SCL renamed /PB8
- net /OLED SDA renamed /PB9
- net /USART_RX renamed /PA3
- net /USART_TX renamed /PA2
- net /tocdodongco1 renamed /PB6
- net /tocdodongco2 renamed /PA6
- net BOOT0 renamed /BOOT0
- net Net-(U1-PC14) renamed /PC14
- net Net-(U1-PC15) renamed /PC15
- D1 pad 1: 3.3V -> +5V
- D1 pad 2: 3.3V -> GND
- D2 pad 1: 3.3V -> /LED1
- D2 pad 2: 3.3V -> unconnected-(D2-A-Pad2)
- U1 pad 1: VBAT -> VDD
- U1 pad 10: /encoderdongco2 -> /PA0
- U1 pad 11: /encoderdongco2 -> /PA1
- U1 pad 14: /INdongco2 -> /PA4
- U1 pad 15: /INdongco2 -> /PA5
- U1 pad 17: unconnected-(U1-PA7-Pad17) -> /PA7
- U1 pad 18: unconnected-(U1-PB0-Pad18) -> /PB0
- U1 pad 19: unconnected-(U1-PB1-Pad19) -> /PB1
- U1 pad 2: unconnected-(U1-PC13-Pad2) -> /PC13
- U1 pad 20: unconnected-(U1-PB2-Pad20) -> /PB2
- U1 pad 21: /MPU6050 SCL -> /PB10
- U1 pad 22: /MPU6050 SCL -> /PB11
- U1 pad 23: 3.3V -> GND
- U1 pad 24: VBAT -> +3.3V
- U1 pad 25: unconnected-(U1-PB12-Pad25) -> /PB12
- U1 pad 26: unconnected-(U1-PB13-Pad26) -> /PB13
- U1 pad 27: unconnected-(U1-PB14-Pad27) -> /PB14
- U1 pad 28: unconnected-(U1-PB15-Pad28) -> /PB15
- U1 pad 29: /encoderdongco1 -> /PA8
- U1 pad 30: /encoderdongco1 -> /PA9
- U1 pad 34: SWDIO -> /PA13
- U1 pad 35: 3.3V -> GND
- U1 pad 36: VBAT -> +3.3V
- U1 pad 37: SCLK -> /PA14
- U1 pad 38: unconnected-(U1-PA15-Pad38) -> /PA15
- U1 pad 39: /INdongco1 -> /PB3
- U1 pad 40: /INdongco1 -> /PB4
- U1 pad 41: unconnected-(U1-PB5-Pad41) -> /PB5
- U1 pad 43: unconnected-(U1-PB7-Pad43) -> /PB7
- U1 pad 47: 3.3V -> GND
- U1 pad 48: VBAT -> +3.3V
- U1 pad 5: unconnected-(U1-PD0-Pad5) -> Net-(U1-PD0)
- U1 pad 6: unconnected-(U1-PD1-Pad6) -> Net-(U1-PD1)
- U1 pad 7: NRST -> /NRST
- U1 pad 8: 3.3V -> GND
- U1 pad 9: VBAT -> Net-(U1-VDDA)
- U6 pad 1: Net-(J1-Pin_1) -> 6-9V Pin lipo
- U6 pad 2: 3.3V -> +5V
- U6 pad 3: 3.3V -> GND
- U6 pad 4: 3.3V -> +5V
- U6 pad 5: 3.3V -> GND
Routing:
- net +5V: track 0.00 -> 143.0 mm
- net +3.3V: track 0.00 -> 117.4 mm
- net 6-9V Pin lipo: track 0.00 -> 16.1 mm
- net GND: track 0.00 -> 1.26 mm

Commit message: cap nhat pcb
Parts:
- removed J1: Conn_01x04_Pin, Connector_PinHeader_2.54mm:PinHeader_1x04_P2.54mm_Vertical
- removed J1: Conn_01x06_Pin, Connector_PinHeader_2.54mm:PinHeader_1x06_P2.54mm_Vertical
- added J3: Conn_01x04_Pin, Connector_PinHeader_2.54mm:PinHeader_1x04_P2.54mm_Vertical, F.Cu at (234.0, 104.5)
- SW2: value SW_Push -> SW_MEC_5E; footprint Button_Switch_THT:SW_PUSH-12mm -> Button_Switch_SMD:SW_MEC_5GSH9
- moved J9 157.5 mm to (248.0, 69.2)
- moved C13 154.4 mm to (253.0, 74.0), turned to -90 degrees
- moved J10 131.0 mm to (134.0, 58.0)
- moved J6 97.0 mm to (171.5, 69.2)
- moved J7 69.2 mm to (203.0, 101.4)
- moved C2 67.0 mm to (160.5, 154.5), turned to 0 degrees
- moved C14 61.2 mm to (154.0, 74.5), turned to 180 degrees
- moved SW1 60.0 mm to (173.0, 120.0)
- moved C17 58.8 mm to (189.5, 124.0), turned to 90 degrees
- moved J8 49.4 mm to (202.5, 140.1), turned to 180 degrees
- moved R6 48.9 mm to (155.0, 83.0), turned to 90 degrees
- moved U6 47.4 mm to (166.0, 162.5)
- moved SW2 46.9 mm to (146.0, 77.5), turned to 180 degrees
- moved J5 41.7 mm to (145.0, 46.0)
- moved C11 35.0 mm to (173.0, 105.3), turned to -90 degrees
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Connections:
- net /PA13 renamed /SWCLK
- net /PA14 renamed /SWDIO
- C10 pad 1: Earth -> GND
- C13 pad 2: /Vcc -> +3.3V
- C14 pad 2: Net-(C14-Pad2) -> /BOOT0
- C5 pad 1: Earth -> GND
- C6 pad 1: Earth -> GND
- C7 pad 1: Earth -> GND
- C8 pad 1: Earth -> GND
- C9 pad 2: Earth -> GND
- D2 pad 2: unconnected-(D2-A-Pad2) -> Net-(D2-A)
- D3 pad 2: unconnected-(D3-A-Pad2) -> Net-(D3-A)
- J10 pad 1: /Vcc -> +3.3V
- J10 pad 3: /C1 -> /C1L
- J10 pad 4: /C2 -> /C2L
- J2 pad 3: /OUT -> /IR1
- J4 pad 3: /OUT -> /IR2
- J5 pad 3: /OUT -> /IR3
- J6 pad 3: /SDA -> /SDA MPU
- J6 pad 4: /SCL -> /SCL MPU
- J7 pad 3: /SDA -> /SDA OLED
- J7 pad 4: /SCK -> /SCK OLED
- J8 pad 3: /IN1 -> /EnB
- J8 pad 4: /IN1 -> /IN4
- J8 pad 5: /IN2 -> /IN3
- J8 pad 7: /tocdo1 -> /IN1
- J8 pad 8: /tocdo2 -> /EnA
- J9 pad 4: /Vcc -> +3.3V
- R5 pad 2: unconnected-(R5-Pad2) -> Net-(D2-A)
- R6 pad 2: Net-(C14-Pad2) -> /BOOT0
- R7 pad 2: unconnected-(R7-Pad2) -> Net-(D3-A)
- SW2 pad 1: GND -> /BOOT0
- SW2 pad 2: Net-(C14-Pad2) -> /BOOT0
- U1 pad 1: VDD -> +3.3V
- U1 pad 10: /PA0 -> /EnB
- U1 pad 11: /PA1 -> /IN4
- U1 pad 12: /PA2 -> /IN3
- U1 pad 13: /PA3 -> /IN2
- U1 pad 14: /PA4 -> /IN1
- U1 pad 15: /PA5 -> /EnA
- U1 pad 16: /PA6 -> unconnected-(U1-PA6-Pad16)
- U1 pad 17: /PA7 -> unconnected-(U1-PA7-Pad17)
- U1 pad 18: /PB0 -> unconnected-(U1-PB0-Pad18)
- U1 pad 19: /PB1 -> unconnected-(U1-PB1-Pad19)
- U1 pad 2: /PC13 -> unconnected-(U1-PC13-Pad2)
- U1 pad 20: /PB2 -> unconnected-(U1-PB2-Pad20)
- U1 pad 21: /PB10 -> /SCK OLED
- U1 pad 22: /PB11 -> /SDA OLED
- U1 pad 25: /PB12 -> unconnected-(U1-PB12-Pad25)
- U1 pad 26: /PB13 -> unconnected-(U1-PB13-Pad26)
- U1 pad 27: /PB14 -> unconnected-(U1-PB14-Pad27)
- U1 pad 28: /PB15 -> unconnected-(U1-PB15-Pad28)
- U1 pad 29: /PA8 -> /C2R
- U1 pad 30: /PA9 -> /C1R
- U1 pad 31: /PA10 -> unconnected-(U1-PA10-Pad31)
- U1 pad 32: /PA11 -> /LED2
- U1 pad 33: /PA12 -> /LED1
- U1 pad 38: /PA15 -> unconnected-(U1-PA15-Pad38)
- U1 pad 39: /PB3 -> /IR1
- U1 pad 40: /PB4 -> /IR2
- U1 pad 41: /PB5 -> /IR3
- U1 pad 42: /PB6 -> /C1L
- U1 pad 43: /PB7 -> /C2L
- U1 pad 45: /PB8 -> /SCL MPU
- U1 pad 46: /PB9 -> /SDA MPU
Routing:
- net +3.3V: track 117.4 -> 335.5 mm
- net /SWDIO: track 0.00 -> 87.5 mm, vias 0 -> 1
- net /IR1: track 0.00 -> 82.3 mm, vias 0 -> 1
- net /SWCLK: track 0.00 -> 81.1 mm, vias 0 -> 1
- net GND: track 1.26 -> 76.8 mm
- net /C2R: track 0.00 -> 65.2 mm, vias 0 -> 1
- net /C1R: track 0.00 -> 64.4 mm, vias 0 -> 1
- net /C1L: track 0.00 -> 57.5 mm, vias 0 -> 1
- net /IR2: track 0.00 -> 55.3 mm, vias 0 -> 1
- net /C2L: track 0.00 -> 54.9 mm, vias 0 -> 1
- net /EnB: track 0.00 -> 54.4 mm, vias 0 -> 1
- net /IR3: track 0.00 -> 52.4 mm, vias 0 -> 1
- net /IN4: track 0.00 -> 51.5 mm, vias 0 -> 1
- net /IN3: track 0.00 -> 48.3 mm, vias 0 -> 1
- net +5V: track 143.0 -> 95.5 mm
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Other:
- board text added: "2K2"

Commit message: LDH_ver1.0
Parts:
- removed C14, C9: 10uF, Capacitor_SMD:C_0603_1608Metric
- removed D1: 1N5822, Diode_THT:D_DO-201AD_P15.24mm_Horizontal
- removed L1: 33uH, Inductor_SMD:L_10.4x10.4_H4.8
- removed SW2: SW_MEC_5E, Button_Switch_SMD:SW_MEC_5GSH9
- removed U6: LM2596S-5, Package_TO_SOT_SMD:TO-263-5_TabPin3
- removed U9: LM1117DT-3.3, Package_TO_SOT_SMD:TO-252-3_TabPin2
- removed Y1: 8MHz, Crystal:Crystal_SMD_HC49-SD_HandSoldering
- added C15: 0.1uF, Capacitor_SMD:C_0603_1608Metric, F.Cu at (197.4, 63.0)
- added C16: 0.1uF, Capacitor_SMD:C_0603_1608Metric, F.Cu at (215.6, 69.7)
- added C24: 22nF, Capacitor_SMD:C_0603_1608Metric, F.Cu at (175.8, 100.5)
- added C25: 22nF, Capacitor_SMD:C_0603_1608Metric, F.Cu at (177.3, 100.5)
- added C26: 22nF, Capacitor_SMD:C_0603_1608Metric, F.Cu at (179.8, 111.4)
- added D4: LED2, LED_SMD:LED_0603_1608Metric_Pad1.05x0.95mm_HandSolder, F.Cu at (216.1, 103.8)
- added D5: 1N5822, Diode_SMD:D_SMA, F.Cu at (184.4, 103.9)
- added J1: Conn_01x04_Pin, Connector_PinHeader_2.54mm:PinHeader_1x04_P2.54mm_Vertical, F.Cu at (225.8, 83.3)
- added J11: Conn_01x02_Pin, Connector_PinHeader_2.54mm:PinHeader_1x02_P2.54mm_Vertical, F.Cu at (177.4, 115.2)
- added J16: USB_C_Receptacle_PowerOnly_6P, Connector_USB:USB_C_Receptacle_GCT_USB4125-xx-x_6P_TopMnt_Horizontal, F.Cu at (205.9, 114.6)
- added L2: 33uH, Inductor_SMD:L_10.4x10.4_H4.8, F.Cu at (188.1, 111.3)
- added R1: 2K2, Resistor_SMD:R_0805_2012Metric_Pad1.20x1.40mm_HandSolder, F.Cu at (218.9, 104.5)
- added R10: 2K2, Resistor_SMD:R_0805_2012Metric_Pad1.20x1.40mm_HandSolder, F.Cu at (176.3, 97.9)
- added R11: 2K2, Resistor_SMD:R_0805_2012Metric_Pad1.20x1.40mm_HandSolder, F.Cu at (181.1, 100.1)
- added R12: 2K2, Resistor_SMD:R_0805_2012Metric_Pad1.20x1.40mm_HandSolder, F.Cu at (179.1, 100.1)
- added R13: 2K2, Resistor_SMD:R_0805_2012Metric_Pad1.20x1.40mm_HandSolder, F.Cu at (176.0, 111.5)
- added R14: 5k1, Resistor_SMD:R_0805_2012Metric_Pad1.20x1.40mm_HandSolder, F.Cu at (197.5, 112.1)
- added R15: 5k1, Resistor_SMD:R_0805_2012Metric_Pad1.20x1.40mm_HandSolder, F.Cu at (199.4, 112.1)
- added R2: 100k, Resistor_SMD:R_0805_2012Metric_Pad1.20x1.40mm_HandSolder, F.Cu at (211.2, 108.2)
- added R8: 2K2, Resistor_SMD:R_0805_2012Metric_Pad1.20x1.40mm_HandSolder, F.Cu at (171.8, 104.9)
- added R9: 2K2, Resistor_SMD:R_0805_2012Metric_Pad1.20x1.40mm_HandSolder, F.Cu at (173.9, 104.9)
- added U2: RT9193-33GB, Package_TO_SOT_SMD:TSOT-23-5, F.Cu at (214.4, 108.0)
- added U3: MP1584, Package_SO:SOIC-8-1EP_3.9x4.9mm_P1.27mm_EP2.29x3mm, F.Cu at (177.8, 106.9)
- added Y2: Crystal_16Mhz, Crystal:Crystal_SMD_2520-4Pin_2.5x2.0mm, F.Cu at (207.6, 72.4)
- C1: value 220uF -> 0.1uF; footprint Capacitor_Tantalum_SMD:CP_EIA-7343-31_Kemet-D_HandSolder -> Capacitor_SMD:C_0603_1608Metric
- C10: value 100nF -> 10uF; footprint Capacitor_SMD:C_0603_1608Metric -> Capacitor_SMD:C_1206_3216Metric
- C13: value 100uF -> 0.1uF
- C17, C7, C8: value 100nF -> 0.1uF
- C19: value 0.1uF -> 1uF
- C2: value 100uF -> 0.1uF; footprint Capacitor_Tantalum_SMD:CP_EIA-6032-28_Kemet-C_HandSolder -> Capacitor_SMD:C_0603_1608Metric
- C3: value 10uF -> 22nF; footprint Capacitor_Tantalum_SMD:CP_EIA-6032-28_Kemet-C_HandSolder -> Capacitor_SMD:C_0603_1608Metric
- C4: value 10uF -> 1uF; footprint Capacitor_Tantalum_SMD:CP_EIA-6032-28_Kemet-C_HandSolder -> Capacitor_SMD:C_0603_1608Metric
- C5, C6: value 100nF -> 22nF
- FB1: footprint Ferrite_THT:LairdTech_28C0236-0JW-10 -> Resistor_SMD:R_0603_1608Metric
- SW1: footprint Button_Switch_THT:SW_PUSH-12mm -> Button_Switch_SMD:SW_Push_SPST_NO_Alps_SKRK
- moved J10 89.7 mm to (215.3, 95.9), turned to 180 degrees
- moved C2 88.8 mm to (208.8, 80.0), turned to 90 degrees
- moved C18 78.8 mm to (223.0, 82.4), turned to 90 degrees
- moved C1 78.1 mm to (208.3, 109.3), turned to 180 degrees
- moved C13 71.3 mm to (181.7, 71.2), turned to 180 degrees
- moved J8 70.2 mm to (172.3, 76.7), turned to 0 degrees
- moved C20 62.6 mm to (210.1, 72.4), turned to -90 degrees
- moved C21 61.1 mm to (207.6, 69.7), turned to 180 degrees
- moved SW1 57.6 mm to (213.7, 79.2), turned to -90 degrees
- moved C3 55.5 mm to (217.5, 108.0), turned to -90 degrees
- moved R6 53.0 mm to (207.4, 91.3), turned to -90 degrees
- moved J9 49.2 mm to (202.9, 88.9), turned to -90 degrees
- moved C17 49.0 mm to (211.1, 80.0)
- moved C6 46.9 mm to (212.7, 103.8), turned to 0 degrees
- moved R3 45.2 mm to (205.4, 74.9), turned to 135 degrees
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Connections:
- net /LED2 renamed /PA11
- C1 pad 1: +5V -> GND
- C1 pad 2: GND -> +5V
- C18 pad 1: GND -> +3.3V
- C18 pad 2: +5V -> GND
- C2 pad 1: 6-9V Pin lipo -> GND
- C2 pad 2: GND -> +3.3V
- C20 pad 2: Net-(U1-PD0) -> /PC14
- C21 pad 2: Net-(U1-PD1) -> /PC15
- C3 pad 1: +5V -> GND
- C3 pad 2: GND -> Net-(U2-~{FLG})
- C4 pad 1: +3.3V -> GND
- C4 pad 2: GND -> +5V
- C5 pad 1: GND -> Net-(D5-K)
- C5 pad 2: +3.3V -> Net-(U3-BST)
- C6 pad 1: GND -> +5V
- C6 pad 2: +3.3V -> GND
- D2 pad 1: /LED1 -> /PA10
- J10 pad 1: +3.3V -> +5V
- J3 pad 1: +3.3V -> +5V
- J6 pad 3: /SDA MPU -> /SDA_MPU
- J6 pad 4: /SCL MPU -> /SCL_MPU
- J7 pad 1: +3.3V -> +5V
- J7 pad 3: /SDA OLED -> /SDA_OLED
- J7 pad 4: /SCK OLED -> /SCL_OLDE
- J9 pad 2: /SWDIO -> /SWCLK
- J9 pad 3: /SWCLK -> /SWDIO
- R3 pad 1: Net-(U1-PD0) -> /PC14
- R3 pad 2: Net-(U1-PD1) -> /PC15
- R6 pad 1: +3.3V -> /BOOT0
- R6 pad 2: /BOOT0 -> GND
- U1 pad 10: /EnB -> unconnected-(U1-PA0-Pad10)
- U1 pad 11: /IN4 -> unconnected-(U1-PA1-Pad11)
- U1 pad 12: /IN3 -> /UART_TX
- U1 pad 13: /IN2 -> /UART_RX
- U1 pad 14: /IN1 -> /IR1
- U1 pad 15: /EnA -> /IR2
- U1 pad 16: unconnected-(U1-PA6-Pad16) -> /IR3
- U1 pad 18: unconnected-(U1-PB0-Pad18) -> /EnA
- U1 pad 19: unconnected-(U1-PB1-Pad19) -> /EnB
- U1 pad 2: unconnected-(U1-PC13-Pad2) -> /PC13
- U1 pad 21: /SCK OLED -> /SCL_MPU
- U1 pad 22: /SDA OLED -> /SDA_MPU
- U1 pad 25: unconnected-(U1-PB12-Pad25) -> /IN4
- U1 pad 26: unconnected-(U1-PB13-Pad26) -> /IN3
- U1 pad 27: unconnected-(U1-PB14-Pad27) -> /IN2
- U1 pad 28: unconnected-(U1-PB15-Pad28) -> /IN1
- U1 pad 31: unconnected-(U1-PA10-Pad31) -> /PA10
- U1 pad 33: /LED1 -> unconnected-(U1-PA12-Pad33)
- U1 pad 34: /SWCLK -> /SWDIO
- U1 pad 37: /SWDIO -> /SWCLK
- U1 pad 39: /IR1 -> unconnected-(U1-PB3-Pad39)
- U1 pad 40: /IR2 -> unconnected-(U1-PB4-Pad40)
- U1 pad 41: /IR3 -> unconnected-(U1-PB5-Pad41)
- U1 pad 42: /C1L -> /SCL_OLDE
- U1 pad 43: /C2L -> /SDA_OLED
- U1 pad 45: /SCL MPU -> /C1L
- U1 pad 46: /SDA MPU -> /C2L
- U1 pad 5: Net-(U1-PD0) -> unconnected-(U1-PD0-Pad5)
- U1 pad 6: Net-(U1-PD1) -> unconnected-(U1-PD1-Pad6)
Routing:
- net +3.3V: track 335.5 -> 212.2 mm, vias 0 -> 5
- net /SWDIO: track 87.5 -> 8.65 mm, vias 1 -> 0
- net /SWCLK: track 81.1 -> 5.55 mm, vias 1 -> 0
- net /IR1: track 82.3 -> 35.1 mm, vias 1 -> 0
- net /C1L: track 57.5 -> 18.1 mm, vias 1 -> 0
- net /C2L: track 54.9 -> 15.7 mm, vias 1 -> 0
- net /UART_RX: track 0.00 -> 39.1 mm
- net /IR2: track 55.3 -> 18.2 mm, vias 1 -> 0
- net /UART_TX: track 0.00 -> 35.9 mm
- net /SCL_MPU: track 0.00 -> 32.8 mm, vias 0 -> 1
- net /SDA_MPU: track 0.00 -> 32.2 mm, vias 0 -> 1
- net /IR3: track 52.4 -> 20.5 mm, vias 1 -> 0
- net /PA10: track 0.00 -> 31.9 mm, vias 0 -> 2
- net /SDA OLED: track 31.3 -> 0.00 mm, vias 1 -> 0
- net /SCK OLED: track 29.9 -> 0.00 mm, vias 1 -> 0
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- added copper zone on F.Cu, net +3.3V
- added copper zone on F.Cu, net +5V
- added copper zone on B.Cu, net GND
- added copper zone on F.Cu, net GND
- added copper zone on F.Cu, net Net-(D5-K)
Other:
- board outline added: 60 x 60.3 mm
- board text added: "3V3"
- board text added: "5V"
- board text added: "C1"
- board text added: "C2"
- board text added: "CLK"
- board text added: "DIO"
- board text added: "EnA"
- board text added: "EnB"
- board text added: "GND"
- board text added: "IN1"
- board text added: "IN2"
- board text added: "IN3"
- board text added: "IN4"
- board text added: "IR"
- board text added: "MPU"
- board text added: "OLED"
- board text added: "SCL"
- board text added: "SDA"
- board text added: "UART_RX"
- board text added: "UART_TX"
- board text removed: "2K2"
