File: micromouse.kicad_sch (KiCad schematic)
At the start: 51 parts, among them J5 Conn_01x03_Pin, J6 Conn_01x03_Pin, M1 Motor_DC, M2 Motor_DC, U1 STM32F103C8Tx, U2 L298N, U3 MPU-6050, U4 LM393, U5 LM393, U6 LM2596S-5, U7 LM393, U9 LM1117DT-3.3, Y1 8MHz

Commit message: Cập nhật schematic
Parts:
- removed C1: 680uF, symbol Device:C
- removed C20: 0.01uF, symbol Device:C
- removed C3: 220uF, symbol Device:C
- removed J5, J6: Conn_01x03_Pin, symbol Connector:Conn_01x03_Pin
- removed M1, M2: Motor_DC, symbol Motor:Motor_DC
- removed R10, R13: 10k, symbol Device:R
- removed R11, R12, R6, R7, R8, R9: R_Variable, symbol Device:R_Variable
- removed R14, R15: 4.7k, symbol Device:R
- removed U2: L298N, Package_TO_SOT_THT:TO-220-15_P2.54x5.08mm_StaggerOdd_Lead4.58mm_Vertical, symbol Driver_Motor:L298N
- removed U3: MPU-6050, Sensor_Motion:InvenSense_QFN-24_4x4mm_P0.5mm, symbol Sensor_Motion:MPU-6050
- removed U4, U5, U7: LM393, symbol Comparator:LM393
- added C1: 220uF, Capacitor_Tantalum_SMD:CP_EIA-7343-31_Kemet-D_HandSolder, symbol Device:C_Polarized
- added C14: 100nF, Capacitor_SMD:C_0603_1608Metric, symbol Device:C
- added C2: 100uF, Capacitor_Tantalum_SMD:CP_EIA-6032-28_Kemet-C_HandSolder, symbol Device:C_Polarized
- added J1, J3: Conn_02x10_Top_Bottom, Connector_PinHeader_2.54mm:PinHeader_2x10_P2.54mm_Vertical_SMD, symbol Connector_Generic:Conn_02x10_Top_Bottom
- added R16: 1.21k, Resistor_SMD:R_0805_2012Metric_Pad1.20x1.40mm_HandSolder, symbol Device:R
- added RV1: variable, Resistor_SMD:R_0805_2012Metric_Pad1.20x1.40mm_HandSolder, symbol Device:R_Potentiometer
- added SW1, SW2: SW_Push, Button_Switch_THT:SW_PUSH-12mm, symbol Switch:SW_Push
- added Y2: 32.768kHz, Crystal:Crystal_SMD_3215-2Pin_3.2x1.5mm, symbol Device:Crystal
- C10: renamed from C12; footprint (none) -> Capacitor_SMD:C_0603_1608Metric
- C11: renamed from C14; footprint (none) -> Capacitor_SMD:C_0603_1608Metric
- C12: renamed from C13; footprint (none) -> Capacitor_SMD:C_0603_1608Metric
- C15: value 100uF -> 8pF; footprint (none) -> Capacitor_SMD:C_0603_1608Metric
- C16: value 0.1uF -> 8pF; footprint (none) -> Capacitor_SMD:C_0603_1608Metric
- C17: value 100uF -> 100nF; footprint (none) -> Capacitor_SMD:C_0603_1608Metric
- C18: value 2200pF -> 0.1uF; footprint (none) -> Capacitor_SMD:C_0603_1608Metric
- C19, C6, C7, C8: footprint (none) -> Capacitor_SMD:C_0603_1608Metric
- C20: renamed from C10; value 330puF -> 22pF; footprint (none) -> Capacitor_SMD:C_0603_1608Metric
- C21: renamed from C9; value 330pF -> 22pF; footprint (none) -> Capacitor_SMD:C_0603_1608Metric
- C3: renamed from C4; footprint (none) -> Capacitor_Tantalum_SMD:CP_EIA-6032-28_Kemet-C_HandSolder
- C4: renamed from C5; footprint (none) -> Capacitor_Tantalum_SMD:CP_EIA-6032-28_Kemet-C_HandSolder
- C5: renamed from C2; footprint (none) -> Capacitor_SMD:C_0603_1608Metric
- C9: renamed from C11; footprint (none) -> Capacitor_SMD:C_0603_1608Metric
- FB1: footprint (none) -> Ferrite_THT:LairdTech_28C0236-0JW-10
- L1: footprint (none) -> Inductor_SMD:L_10.4x10.4_H4.8
- R1, R2: footprint (none) -> Resistor_SMD:R_0805_2012Metric_Pad1.20x1.40mm_HandSolder
- R3: value 0.5 -> 1M; footprint (none) -> Resistor_SMD:R_0805_2012Metric_Pad1.20x1.40mm_HandSolder
- R4: value 0.5 -> 10K; footprint (none) -> Resistor_SMD:R_0805_2012Metric_Pad1.20x1.40mm_HandSolder
- R5: value 10k -> 100K; footprint (none) -> Resistor_SMD:R_0805_2012Metric_Pad1.20x1.40mm_HandSolder
- Y1: footprint (none) -> Crystal:Crystal_SMD_HC49-SD_HandSoldering
Connections:
- net REGOUT is gone; now on net GND: C19.1
- net +3.3V: now also C19.2, R4.1, J3.18 (Pin_18), J3.8 (Pin_8), SW2.1; no longer C16.2, R5.1, U1.1 (VBAT)
- net +5V: now also C18.2; no longer C15.2, C17.2
- net 5V: now also C1.1, RV1.1; no longer U6.4 (FB)
- net 6-9V Pin lipo: now also C2.1
- net BOOT0: now also R5.1, C14.2, SW2.2
- net GND: now also C11.1, C12.1, C18.1, R5.2, C1.2, C14.1, C2.2, J3.19 (Pin_19), J3.9 (Pin_9), R16.2, SW1.2; no longer C18.2, C19.2, R3.2, R4.2
- net NRST: now also C17.2, R4.2, J3.17 (Pin_17), SW1.1
- net PA0: now also J1.11 (Pin_11)
- net PA1: now also J1.12 (Pin_12)
- net PA10: now also J3.11 (Pin_11); no longer R5.2
- net PA11: now also J3.12 (Pin_12)
- net PA12: now also J3.13 (Pin_13)
- net PA4: now also J1.15 (Pin_15)
- net PA5: now also J1.16 (Pin_16)
- net PA6: now also J1.17 (Pin_17)
- net PA8: now also J1.19 (Pin_19)
- net PA9: now also J1.20 (Pin_20)
- net PB10: now also J3.1 (Pin_1); no longer U1.22 (PB11)
- net PB3: now also J1.4 (Pin_4)
- net PB4: now also J1.5 (Pin_5)
- net PB5: now also J1.6 (Pin_6)
- net PB6: now also J1.7 (Pin_7)
- net at C20.2, Y1.1: now also R3.1, U1.5 (PD0); no longer U1.3 (PC14)
- net at C21.2, Y1.2: now also R3.2, U1.6 (PD1); no longer U1.4 (PC15)
- net PA2: now reaches U1.12 (PA2)
- net PA2: now also J1.13 (Pin_13)
- net PA3: now reaches U1.13 (PA3)
- net PA3: now also J1.14 (Pin_14)
- net PA7: now reaches U1.17 (PA7)
- net PA7: now also J1.18 (Pin_18)
- net PB0: now reaches U1.18 (PB0)
- net PB0: now also J1.1 (Pin_1)
- net PB1: now reaches U1.19 (PB1)
- net PB1: now also J1.2 (Pin_2)
- net PC13: now reaches U1.2 (PC13)
- net PC13: now also J3.10 (Pin_10)
- net PB2: now reaches U1.20 (PB2)
- net PB2: now also J1.3 (Pin_3)
- net PB12: now reaches U1.25 (PB12)
- net PB12: now also J3.3 (Pin_3)
- net PB13: now reaches U1.26 (PB13)
- net PB13: now also J3.4 (Pin_4)
- net PB14: now reaches U1.27 (PB14)
- net PB14: now also J3.5 (Pin_5)
- net PB15: now reaches U1.28 (PB15)
- net PB15: now also J3.6 (Pin_6)
- net PA15: now reaches U1.38 (PA15)
- net PA15: now also J3.16 (Pin_16)
- net PB7: now reaches U1.43 (PB7)
- net PB7: now also J1.8 (Pin_8)
- net PB8: now reaches U1.45 (PB8)
- net PB8: now also J1.9 (Pin_9)
- net PB9: now reaches U1.46 (PB9)
- net PB9: now also J1.10 (Pin_10)
- net SCLK renamed PA14
- net PA14: now also J3.15 (Pin_15)
- net SWDIO renamed PA13
- net PA13: now also J3.14 (Pin_14)
- new net: R16.1, RV1.2, RV1.3, U6.4 (FB)
- new net PB11: J3.2 (Pin_2), U1.22 (PB11)
- new net PC14: C16.2, U1.3 (PC14), Y2.1
- new net PC15: C15.2, U1.4 (PC15), Y2.2
- new net VDD: J3.7 (Pin_7), U1.1 (VBAT)
Other:
- note removed: "KHOI DRIVER"
- note removed: "KHOI GIA TOC"
- note removed: "KHOI IR"
- moved on the sheet: C20, C21, Y1

Commit message: cap nhat schematic
Parts:
- removed J1, J3: Conn_02x10_Top_Bottom, Connector_PinHeader_2.54mm:PinHeader_2x10_P2.54mm_Vertical_SMD, symbol Connector_Generic:Conn_02x10_Top_Bottom
- removed SW2: SW_Push, Button_Switch_THT:SW_PUSH-12mm, symbol Switch:SW_Push
- added C13: 100uF, Capacitor_SMD:C_0603_1608Metric, symbol Device:C
- added D2: LED1, LED_SMD:LED_0603_1608Metric_Pad1.05x0.95mm_HandSolder, symbol Device:LED
- added D3: LED2, LED_SMD:LED_0603_1608Metric_Pad1.05x0.95mm_HandSolder, symbol Device:LED
- added J1: Conn_01x06_Pin, Connector_PinHeader_2.54mm:PinHeader_1x06_P2.54mm_Vertical, symbol Connector:Conn_01x06_Pin
- added J2, J4, J5: Conn_01x03_Pin, Connector_PinHeader_2.54mm:PinHeader_1x03_P2.54mm_Vertical, symbol Connector:Conn_01x03_Pin
- added J6, J7: Conn_01x04_Pin, Connector_PinHeader_2.54mm:PinHeader_1x04_P2.54mm_Vertical, symbol Connector:Conn_01x04_Pin
- added J8: Conn_01x08_Pin, Connector_PinHeader_2.54mm:PinHeader_1x08_P2.54mm_Vertical, symbol Connector:Conn_01x08_Pin
- added J9: Conn_01x04, Connector_PinHeader_2.54mm:PinHeader_1x04_P2.54mm_Vertical, symbol Connector_Generic:Conn_01x04
- added R6: 10K, Resistor_SMD:R_0805_2012Metric_Pad1.20x1.40mm_HandSolder, symbol Device:R
- added R7: 2K2, Resistor_SMD:R_0805_2012Metric_Pad1.20x1.40mm_HandSolder, symbol Device:R
- added SW3: SW_DP3T, Button_Switch_SMD:SW_SPST_B3U-1000P, symbol Switch:SW_DP3T
- C14: value 100nF -> 10uF
- R5: value 100K -> 2K2
Connections:
- net +3.3V: now also R5.1, J2.1 (Pin_1), J4.1 (Pin_1), J5.1 (Pin_1), J6.1 (Pin_1), J7.1 (Pin_1), R6.1, R7.1
- net +5V: now also J8.1 (Pin_1)
- net BOOT0: no longer C14.2, R5.1
- net GND: now also C13.1, J1.2 (Pin_2), J2.2 (Pin_2), J4.2 (Pin_2), J5.2 (Pin_2), J6.2 (Pin_2), J7.2 (Pin_2), J8.2 (Pin_2), J9.1 (Pin_1), SW3.3, SW3.4; no longer R5.2
- net PA13: now also J9.3 (Pin_3)
- net PA14: now also J9.2 (Pin_2)
- new net: C14.2, R6.2, SW3.1, SW3.2
- new net C1: J1.3 (Pin_3), J1.4 (Pin_4)
- new net C2: J1.5 (Pin_5), J1.6 (Pin_6)
- new net IN1: J8.3 (Pin_3), J8.4 (Pin_4)
- new net IN2: J8.5 (Pin_5), J8.6 (Pin_6)
- new net LED1: D2.1 (K)
- new net LED2: D3.1 (K)
- new net OUT: J2.3 (Pin_3), J4.3 (Pin_3), J5.3 (Pin_3)
- new net SCK: J7.4 (Pin_4)
- new net SCL: J6.4 (Pin_4)
- new net SDA: J6.3 (Pin_3), J7.3 (Pin_3)
- new net Vcc: C13.2, J1.1 (Pin_1), J9.4 (Pin_4)
- new net tocdo1: J8.7 (Pin_7)
- new net tocdo2: J8.8 (Pin_8)
Other:
- note added: "BOOT0"
- note added: "Chân encoder"
- note added: "Chân nạp code"
- note added: "Chân nối IR"
- note added: "Chân nối MPU"
- note added: "Chân nối OLED"
- note added: "Chân nối driver"
- note added: "Thạch anh phụ"
- moved on the sheet: C14, C15, C16, R5, Y2

Commit message: cap nhat pcb
Parts:
- removed C15, C16: 8pF, Capacitor_SMD:C_0603_1608Metric, symbol Device:C
- removed J1: Conn_01x06_Pin, Connector_PinHeader_2.54mm:PinHeader_1x06_P2.54mm_Vertical, symbol Connector:Conn_01x06_Pin
- removed R1: 121, Resistor_SMD:R_0805_2012Metric_Pad1.20x1.40mm_HandSolder, symbol Device:R
- removed R16: 1.21k, Resistor_SMD:R_0805_2012Metric_Pad1.20x1.40mm_HandSolder, symbol Device:R
- removed R2: 196, Resistor_SMD:R_0805_2012Metric_Pad1.20x1.40mm_HandSolder, symbol Device:R
- removed RV1: variable, Resistor_SMD:R_0805_2012Metric_Pad1.20x1.40mm_HandSolder, symbol Device:R_Potentiometer
- removed SW3: SW_DP3T, Button_Switch_SMD:SW_SPST_B3U-1000P, symbol Switch:SW_DP3T
- removed Y2: 32.768kHz, Crystal:Crystal_SMD_3215-2Pin_3.2x1.5mm, symbol Device:Crystal
- added J10, J3: Conn_01x04_Pin, Connector_PinHeader_2.54mm:PinHeader_1x04_P2.54mm_Vertical, symbol Connector:Conn_01x04_Pin
- added SW2: SW_MEC_5E, Button_Switch_SMD:SW_MEC_5GSH9, symbol Switch:SW_MEC_5E
- C10, C5, C6, C7, C8: value 100uF -> 100nF
Connections:
- net 5V is gone; now on net +5V: C1.1, D1.1 (K), L1.1, L1.2, U6.2 (OUT)
- net LED1 is gone; now on net PA11: D2.1 (K)
- net LED2 is gone; now on net PA12: D3.1 (K)
- net VDD is gone; now on net +3.3V: U1.1 (VBAT)
- net +5V: now also U6.4 (FB)
- net BOOT0: now also C14.2, R6.2, SW2.1, SW2.2
- net C1: now also J10.3 (Pin_3), J3.3 (Pin_3)
- net C2: now also J10.4 (Pin_4), J3.4 (Pin_4)
- net GND: now also U9.1 (GND), J10.2 (Pin_2), J3.2 (Pin_2), SW2.3 (K), SW2.4 (A)
- net Vcc: now also J10.1 (Pin_1), J3.1 (Pin_1)
- net at D2.2 (A): now also R5.2
- net at R7.2: now also D3.2 (A)
Other:
- note added: "Chân pin lipo"
- note removed: "Thạch anh phụ"
- moved on the sheet: C19, C4, D2, D3, R6

Commit message: cap nhat pcb
Connections:
- net PA3 is gone; now on net IN2: U1.13 (PA3)
- net PA4 is gone; now on net IN1: U1.14 (PA4)
- net PB10 is gone; now on net SCK: U1.21 (PB10)
- net PB11 is gone; now on net SDA: U1.22 (PB11)
- net PB6 is gone; now on net C1L: U1.42 (PB6)
- net PB7 is gone; now on net C2L: U1.43 (PB7)
- net PB8 is gone; now on net SCL: U1.45 (PB8)
- net PB9 is gone; now on net SDA: U1.46 (PB9)
- net Vcc is gone; now on net +3.3V: C13.2, J10.1 (Pin_1), J3.1 (Pin_1), J9.4 (Pin_4)
- net tocdo1 is gone; now on net IN1: J8.7 (Pin_7)
- net tocdo2 is gone; now on net EnA: J8.8 (Pin_8)
- net IN1: no longer J8.3 (Pin_3), J8.4 (Pin_4)
- net IN2: no longer J8.5 (Pin_5)
- net PA11: no longer U1.32 (PA11)
- net PA12: no longer U1.33 (PA12)
- net C1 renamed C1L
- net C1L: no longer J3.3 (Pin_3)
- net C2 renamed C2L
- net C2L: no longer J3.4 (Pin_4)
- removed net OUT: J2.3 (Pin_3), J4.3 (Pin_3), J5.3 (Pin_3)
- net PA0 renamed EnB
- net EnB: now also J8.3 (Pin_3)
- net PA1 renamed IN4
- net IN4: now also J8.4 (Pin_4)
- net PA10: no longer names the net of U1.31 (PA10)
- net PA13: no longer names the net of J9.3 (Pin_3)
- net PA13: no longer U1.34 (PA13)
- net PA14: no longer names the net of J9.2 (Pin_2)
- net PA14: no longer U1.37 (PA14)
- net PA15: no longer names the net of U1.38 (PA15)
- net PA2 renamed IN3
- net IN3: now also J8.5 (Pin_5)
- net PA5 renamed EnA
- net PA6: no longer names the net of U1.16 (PA6)
- net PA7: no longer names the net of U1.17 (PA7)
- net PA8 renamed C2R
- net C2R: now also J3.4 (Pin_4)
- net PA9 renamed C1R
- net C1R: now also J3.3 (Pin_3)
- net PB0: no longer names the net of U1.18 (PB0)
- net PB1: no longer names the net of U1.19 (PB1)
- net PB12: no longer names the net of U1.25 (PB12)
- net PB13: no longer names the net of U1.26 (PB13)
- net PB14: no longer names the net of U1.27 (PB14)
- net PB15: no longer names the net of U1.28 (PB15)
- net PB2: no longer names the net of U1.20 (PB2)
- net PB3 renamed IR1
- net IR1: now also J2.3 (Pin_3)
- net PB4 renamed IR2
- net IR2: now also J4.3 (Pin_3)
- net PB5 renamed IR3
- net IR3: now also J5.3 (Pin_3)
Other:
- moved on the sheet: SW1

Commit message: LDH_ver1.0
Parts:
- removed C1: 220uF, Capacitor_Tantalum_SMD:CP_EIA-7343-31_Kemet-D_HandSolder, symbol Device:C_Polarized
- removed C14, C9: 10uF, Capacitor_SMD:C_0603_1608Metric, symbol Device:C
- removed C2: 100uF, Capacitor_Tantalum_SMD:CP_EIA-6032-28_Kemet-C_HandSolder, symbol Device:C_Polarized
- removed C3, C4: 10uF, Capacitor_Tantalum_SMD:CP_EIA-6032-28_Kemet-C_HandSolder, symbol Device:C_Polarized
- removed D1: 1N5822, Diode_THT:D_DO-201AD_P15.24mm_Horizontal, symbol Diode:1N5822
- removed L1: 33uH, Inductor_SMD:L_10.4x10.4_H4.8, symbol Device:L
- removed SW2: SW_MEC_5E, Button_Switch_SMD:SW_MEC_5GSH9, symbol Switch:SW_MEC_5E
- removed U6: LM2596S-5, Package_TO_SOT_SMD:TO-263-5_TabPin3, symbol Regulator_Switching:LM2596S-5
- removed U9: LM1117DT-3.3, Package_TO_SOT_SMD:TO-252-3_TabPin2, symbol Regulator_Linear:LM1117DT-3.3
- removed Y1: 8MHz, Crystal:Crystal_SMD_HC49-SD_HandSoldering, symbol Device:Crystal
- added C1, C15, C16, C2: 0.1uF, Capacitor_SMD:C_0603_1608Metric, symbol Device:C
- added C24, C25, C26, C3: 22nF, Capacitor_SMD:C_0603_1608Metric, symbol Device:C
- added C4: 1uF, Capacitor_SMD:C_0603_1608Metric, symbol Device:C
- added D4: LED2, LED_SMD:LED_0603_1608Metric_Pad1.05x0.95mm_HandSolder, symbol Device:LED
- added D5: 1N5822, Diode_SMD:D_SMA, symbol Diode:1N5822
- added J1: Conn_01x04_Pin, Connector_PinHeader_2.54mm:PinHeader_1x04_P2.54mm_Vertical, symbol Connector:Conn_01x04_Pin
- added J11: Conn_01x02_Pin, Connector_PinHeader_2.54mm:PinHeader_1x02_P2.54mm_Vertical, symbol Connector:Conn_01x02_Pin
- added J16: USB_C_Receptacle_PowerOnly_6P, Connector_USB:USB_C_Receptacle_GCT_USB4125-xx-x_6P_TopMnt_Horizontal, symbol Connector:USB_C_Receptacle_PowerOnly_6P
- added L2: 33uH, Inductor_SMD:L_10.4x10.4_H4.8, symbol Device:L
- added R1, R10, R11, R12, R13, R8, R9: 2K2, Resistor_SMD:R_0805_2012Metric_Pad1.20x1.40mm_HandSolder, symbol Device:R
- added R14, R15: 5k1, Resistor_SMD:R_0805_2012Metric_Pad1.20x1.40mm_HandSolder, symbol Device:R
- added R2: 100k, Resistor_SMD:R_0805_2012Metric_Pad1.20x1.40mm_HandSolder, symbol Device:R
- added U2: RT9193-33GB, Package_TO_SOT_SMD:TSOT-23-5, symbol Power_Management:RT9742ANGJ5F
- added U3: MP1584, Package_SO:SOIC-8-1EP_3.9x4.9mm_P1.27mm_EP2.29x3mm, symbol Regulator_Switching:ADP2303ARDZ-5.0
- added Y2: Crystal_16Mhz, Crystal:Crystal_SMD_2520-4Pin_2.5x2.0mm, symbol Device:Crystal_GND24
- C10: value 100nF -> 10uF; footprint Capacitor_SMD:C_0603_1608Metric -> Capacitor_SMD:C_1206_3216Metric
- C13: value 100uF -> 0.1uF
- C17, C7, C8: value 100nF -> 0.1uF
- C19: value 0.1uF -> 1uF
- C5, C6: value 100nF -> 22nF
- FB1: footprint Ferrite_THT:LairdTech_28C0236-0JW-10 -> Resistor_SMD:R_0603_1608Metric
- SW1: footprint Button_Switch_THT:SW_PUSH-12mm -> Button_Switch_SMD:SW_Push_SPST_NO_Alps_SKRK
Connections:
- net PA12 is gone; now on net PA11: D3.1 (K)
- net +3.3V: now also C18.1, C15.2, C16.2, C2.2, J1.1 (Pin_1), R1.1, U2.5 (VOUT); no longer C5.2, C6.2, J10.1 (Pin_1), J3.1 (Pin_1), J7.1 (Pin_1), R6.1
- net +5V: now also C6.1, J10.1 (Pin_1), J3.1 (Pin_1), J7.1 (Pin_1), C1.2, C4.2, J16.A9 (VBUS), J16.B9 (VBUS), L2.2, R2.1, R8.2, U2.1 (VIN); no longer C18.2
- net BOOT0: now also R6.1; no longer R6.2
- net C1L: now also U1.45 (PB8); no longer U1.42 (PB6)
- net C2L: now also U1.46 (PB9); no longer U1.43 (PB7)
- net EnA: now also U1.18 (PB0); no longer U1.15 (PA5)
- net EnB: now also U1.19 (PB1); no longer U1.10 (PA0)
- net GND: now also C10.1, C18.2, C6.2, C7.1, C8.1, R6.2, C1.1, C15.1, C16.1, C2.1, C25.2, C26.2, C3.1, C4.1, D4.1 (K), D5.2 (A), J1.2 (Pin_2), J11.2 (Pin_2), J16.A12 (GND), J16.B12 (GND), J16.S1 (SHIELD), R10.2, R12.2, R13.2, R14.2, R15.2, R9.2, U2.2 (GND), U3.5 (GND), U3.9 (PADGND), Y2.2, Y2.4; no longer C18.1
- net IN1: now also U1.28 (PB15); no longer U1.14 (PA4)
- net IN2: now also U1.27 (PB14); no longer U1.13 (PA3)
- net IN3: now also U1.26 (PB13); no longer U1.12 (PA2)
- net IN4: now also U1.25 (PB12); no longer U1.11 (PA1)
- net IR1: now also U1.14 (PA4); no longer U1.39 (PB3)
- net IR2: now also U1.15 (PA5); no longer U1.40 (PB4)
- net IR3: now also U1.16 (PA6); no longer U1.41 (PB5)
- net PA11: now also U1.32 (PA11); no longer D2.1 (K)
- net PC14: now also C20.2, R3.1, Y2.3
- net PC15: now also C21.2, R3.2, Y2.1
- net SWCLK: now reaches J9.2 (Pin_2)
- net SWCLK: now also U1.37 (PA14)
- net SWDIO: now reaches J9.3 (Pin_3)
- net SWDIO: now also U1.34 (PA13)
- net PA10: now reaches U1.31 (PA10)
- net PA10: now also D2.1 (K)
- removed net Earth: C10.1, C5.1, C6.1, C7.1, C8.1
- net SCK renamed SCL_MPU
- net SCL_MPU: now also J6.4 (Pin_4); no longer J7.4 (Pin_4)
- removed net SCL: J6.4 (Pin_4), U1.45 (PB8)
- net SDA renamed SDA_MPU
- net SDA_MPU: no longer J7.3 (Pin_3), U1.46 (PB9)
- new net: R11.2, R12.1, U3.2 (EN)
- new net: R2.2, U2.3 (EN)
- new net: D4.2 (A), R1.2
- new net: J16.A5 (CC1), R15.1
- new net: C5.1, D5.1 (K), L2.1, U3.1 (SW)
- new net: C5.2, U3.8 (BST)
- new net: C3.2, U2.4 (~{FLG})
- new net: J16.B5 (CC2), R14.1
- new net: R8.1, R9.1, U3.4 (FB)
- new net: C24.1, C25.1, U3.3 (COMP)
- new net: C24.2, R10.1
- new net: R13.1, U3.6 (NC)
- new net SCL_OLDE: J7.4 (Pin_4), U1.42 (PB6)
- new net SDA_OLED: J7.3 (Pin_3), U1.43 (PB7)
- new net UART_RX: J1.4 (Pin_4), U1.13 (PA3)
- new net UART_TX: J1.3 (Pin_3), U1.12 (PA2)
- new net Vin: C26.1, J11.1 (Pin_1), R11.1, U3.7 (Vin)
- now unconnected: U1.5 (PD0), U1.6 (PD1)
Other:
- note added: "UART"
- note removed: "BOOT0"
- moved on the sheet: C17, C19, C20, C21, C7, C8, D2, D3, J10, J3, R3, R4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
